File: PROG/PROG_for_DEVil-KIT.kicad_pcb (KiCad board)
At the start: 2 copper layers, 15.5 x 35.7 mm, 27 parts, among them J1 POWER, J2 PROG, Q1 BSS138LT1G, Q2 BSS138LT1G, Q3 BSS138LT1G, U1 AMS1117-3.3

Commit message: Add files via upload
Parts:
- removed R2, R4: 10k, Resistor_SMD:R_0603_1608Metric_Pad1.05x0.95mm_HandSolder
- removed mQ4: BSS138LT1G, Package_TO_SOT_SMD:SOT-323_SC-70
- added Q4: BSS138LT1G, Package_TO_SOT_SMD:SOT-323_SC-70, B.Cu at (71.1, 40.8)
- R1, R3, R5, R7: value 4.7k -> 10k
- moved R3 6.68 mm to (73.4, 38.7), turned to 270 degrees
- moved R5 5.12 mm to (78.0, 37.4), turned to 90 degrees
- moved R1 4.16 mm to (73.8, 46.6), turned to 90 degrees
- moved C1 3.95 mm to (70.2, 43.0)
- moved R8 3.14 mm to (73.9, 44.1), turned to 0 degrees
- moved C4 1.88 mm to (74.2, 42.5), turned to 0 degrees
- moved C3 1.21 mm to (75.2, 35.5), turned to 0 degrees
- moved R6 1.17 mm to (75.2, 34.0), turned to 0 degrees
- moved C2 0.98 mm to (71.8, 34.1), turned to 90 degrees
- moved R7 0.58 mm to (70.1, 39.1)
- moved Q1 0.30 mm to (71.3, 45.7)
Connections:
- C4 pad 2: RX -> RX_PROG
- C5 pad 2: Net-(C5-Pad2) -> GND
- C6 pad 2: Net-(C5-Pad2) -> GND
- Q1 pad 1: RST -> +3V3
- Q1 pad 3: GND -> RST
- Q2 pad 1: BOOT -> +3V3
- Q2 pad 3: GND -> BOOT
- Q3 pad 1: TX -> +3V3
- Q3 pad 3: GND -> TX
- R1 pad 1: RST_PROG -> RST
- R3 pad 1: BOOT_PROG -> BOOT
- R5 pad 1: TX_PROG -> TX
- R6 pad 1: TX -> +3V3
- R6 pad 2: GND -> TX_PROG
- R8 pad 1: RX_PROG -> +3V3
- R8 pad 2: GND -> RX_PROG
- U1 pad 1: Net-(C5-Pad2) -> GND
Routing:
- net GND: track 94.4 -> 121.8 mm, vias 14 -> 20
- net +3V3: track 31.3 -> 52.1 mm, vias 3 -> 5
- net Net-(C5-Pad2): track 15.7 -> 0.00 mm, vias 2 -> 0
- net RST_PROG: track 25.3 -> 20.0 mm
- net TX: track 31.4 -> 26.5 mm
- net RX: track 27.4 -> 23.5 mm
- net (no net): track 0.00 -> 3.88 mm
- net BOOT_PROG: track 49.7 -> 46.9 mm
- net RST: track 13.3 -> 11.4 mm
- net RX_PROG: track 41.7 -> 43.0 mm
- net BOOT: track 30.3 -> 29.1 mm
- net 5V_PROG: track 33.1 -> 32.1 mm
- net TX_PROG: track 48.8 -> 48.1 mm
- net Net-(C6-Pad1): vias 1 -> 2
Other:
- outline, holes or cut-outs redrawn

Commit message: Add files via upload
Parts:
- added G***: LOGO, PCB_lib:pcb_logo_devil_sm, F.Cu at (73.2, 62.5)
